File: Schematics/MainBoard/MainBoard.kicad_pcb (KiCad board)
At the start: 4 copper layers, 175 x 160 mm, 258 parts, among them IC1 ATF1508AS-7AX100, IC2 MP2636GR-P, IC3 W65C22S6TQG-14, J1 Conn_02x05_Odd_Even, J10 Conn_02x05_Odd_Even, J11 Conn_02x04_Odd_Even, J12 Conn_02x06_Odd_Even, J13 Conn_02x06_Odd_Even, J14 KeyConn, J15 Conn_01x06, J16 Conn_01x03, J18 Conn_01x03, J2 USBPD_PROG, J3 USB_C_Receptacle_USB2.0_16P, J4 BATTERY JST PH-2A, J5 Conn_02x20_Odd_Even, J6 AudioJack3, J7 Conn_01x02, J8 Conn_02x26_Top_Bottom, J9 DIN41612_02x32_AC, Q1 STL9P3LLH6, Q2 IRLML6402, Q3 STL9P3LLH6, U1 TC1232, U10 FT245RNL, U11 LM386, U12 W65C51NxP, U13 ESP8266-01_ESP-01, U14 AMS1117-3.3, U15 TXS0102DCT, U16 ATmega644P-20A, U2 W65C02S6TQG-14, U3 IS62C256AL, U4 IS62C256AL, U5 SST39SF010, U6 STUSB4500QTR, U7 AP63203WU, U8 TXS0108, U9 TXS0108, X1 16MHz, X2 1.8432MHz, Y1 ECS-3961-200-AU-TR

Commit message: Updated USB wiring, moved key parts, increased board dimensions
Parts:
- C56, C57, C58, C59, J12, J13, J14, J3, J5, J6, LS1, S1, S2, U13, VR1, X1, X2: moved to B.Cu
- moved C48 422.2 mm to (48.8, 153.2)
- moved C49 422.2 mm to (48.8, 155.7)
- moved D17 422.2 mm to (48.4, 150.2)
- moved R82 422.2 mm to (48.3, 158.0)
- moved U12 422.2 mm to (30.0, 124.0)
- moved X2 412.6 mm to (60.5, 132.6), turned to 180 degrees
- moved C55 350.8 mm to (35.5, 65.0)
- moved U11 350.8 mm to (24.3, 60.7)
- moved C45 350.8 mm to (35.5, 59.9)
- moved C46 350.8 mm to (35.5, 62.5)
- moved C54 350.8 mm to (54.5, 46.4)
- moved C56 350.8 mm to (47.6, 64.5), turned to 180 degrees
- moved LS1 350.8 mm to (46.3, 48.4), turned to 180 degrees
- moved R85 350.8 mm to (53.8, 39.9)
- moved R86 350.8 mm to (54.5, 49.3)
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Other:
- board size 175 x 160 mm -> 190 x 175 mm

Commit message: rough placement of parts to help with 3D CAD
Parts:
- removed C67, C68, C69: 100nF, Capacitor_SMD:C_0402_1005Metric
- removed J14: KeyConn, Connector_PinHeader_2.54mm:PinHeader_1x04_P2.54mm_Horizontal
- removed J15: Conn_01x06, Connector_PinHeader_1.00mm:PinHeader_1x06_P1.00mm_Vertical_SMD_Pin1Left
- removed J9: DIN41612_02x32_AC, Connector_DIN:DIN41612_R_2x32_Female_Horizontal_THT
- removed R19, R20, R23: 3K3, Resistor_SMD:R_0402_1005Metric
- removed U16: ATmega644P-20A, Package_QFP:TQFP-44_10x10mm_P0.8mm
- removed X2: 1.8432MHz, Oscillator:Oscillator_DIP-8
- added C37: 100nF, Capacitor_SMD:C_0805_2012Metric, F.Cu at (119.1, 374.8)
- added D1: 1N4148W, Diode_SMD:D_SOD-123, F.Cu at (209.4, 370.1)
- added D15: 1N4148W, Diode_SMD:D_SOD-123, F.Cu at (209.4, 383.4)
- added D20: 1N4148W, Diode_SMD:D_SOD-123, F.Cu at (209.4, 386.8)
- added D22: 1N4148W, Diode_SMD:D_SOD-123, F.Cu at (209.4, 390.1)
- added D23: 1N4148W, Diode_SMD:D_SOD-123, F.Cu at (209.4, 393.5)
- added D24: 1N4148W, Diode_SMD:D_SOD-123, F.Cu at (209.4, 396.9)
- added D25: 1N4148W, Diode_SMD:D_SOD-123, F.Cu at (209.4, 400.2)
- added D26: 1N4148W, Diode_SMD:D_SOD-123, F.Cu at (209.4, 403.6)
- added D27: 1N4148W, Diode_SMD:D_SOD-123, F.Cu at (209.4, 406.9)
- added D28: 1N4148W, Diode_SMD:D_SOD-123, F.Cu at (215.2, 370.1)
- added D29: 1N4148W, Diode_SMD:D_SOD-123, F.Cu at (215.2, 373.4)
- added D30: 1N4148W, Diode_SMD:D_SOD-123, F.Cu at (215.2, 376.8)
- added D31: 1N4148W, Diode_SMD:D_SOD-123, F.Cu at (215.2, 380.1)
- added D32: 1N4148W, Diode_SMD:D_SOD-123, F.Cu at (215.2, 383.4)
- added D33: 1N4148W, Diode_SMD:D_SOD-123, F.Cu at (215.2, 386.8)
- added D34: 1N4148W, Diode_SMD:D_SOD-123, F.Cu at (215.2, 390.1)
- added D35: 1N4148W, Diode_SMD:D_SOD-123, F.Cu at (215.2, 393.5)
- added D36: 1N4148W, Diode_SMD:D_SOD-123, F.Cu at (215.2, 396.9)
- added D37: 1N4148W, Diode_SMD:D_SOD-123, F.Cu at (215.2, 400.2)
- added D38: 1N4148W, Diode_SMD:D_SOD-123, F.Cu at (215.2, 403.6)
- added D39: 1N4148W, Diode_SMD:D_SOD-123, F.Cu at (215.2, 406.9)
- added D40: 1N4148W, Diode_SMD:D_SOD-123, F.Cu at (221.0, 370.1)
- added D41: 1N4148W, Diode_SMD:D_SOD-123, F.Cu at (221.0, 373.4)
- added D42: 1N4148W, Diode_SMD:D_SOD-123, F.Cu at (221.0, 376.8)
- added D43: 1N4148W, Diode_SMD:D_SOD-123, F.Cu at (221.0, 380.1)
- added D44: 1N4148W, Diode_SMD:D_SOD-123, F.Cu at (221.0, 383.4)
- added D45: 1N4148W, Diode_SMD:D_SOD-123, F.Cu at (221.0, 386.8)
- added D46: 1N4148W, Diode_SMD:D_SOD-123, F.Cu at (221.0, 390.1)
- added D47: 1N4148W, Diode_SMD:D_SOD-123, F.Cu at (221.0, 393.5)
- added D48: 1N4148W, Diode_SMD:D_SOD-123, F.Cu at (221.0, 396.9)
- added D49: 1N4148W, Diode_SMD:D_SOD-123, F.Cu at (221.0, 400.2)
- added D50: 1N4148W, Diode_SMD:D_SOD-123, F.Cu at (221.0, 403.6)
- added D51: 1N4148W, Diode_SMD:D_SOD-123, F.Cu at (221.0, 406.9)
- added D52: 1N4148W, Diode_SMD:D_SOD-123, F.Cu at (226.8, 370.1)
- added D53: 1N4148W, Diode_SMD:D_SOD-123, F.Cu at (226.8, 373.4)
- added D54: 1N4148W, Diode_SMD:D_SOD-123, F.Cu at (226.8, 376.8)
- added D55: 1N4148W, Diode_SMD:D_SOD-123, F.Cu at (226.8, 380.1)
- added D56: LED, LED_SMD:LED_0603_1608Metric, F.Cu at (311.4, 371.7)
- added D57: 1N4148W, Diode_SMD:D_SOD-123, F.Cu at (226.8, 383.4)
- added D58: 1N4148W, Diode_SMD:D_SOD-123, F.Cu at (226.8, 386.8)
- added D59: 1N4148W, Diode_SMD:D_SOD-123, F.Cu at (226.8, 390.1)
- added D60: LED, LED_SMD:LED_0603_1608Metric, F.Cu at (311.4, 374.3)
- added D61: LED, LED_SMD:LED_0603_1608Metric, F.Cu at (311.4, 376.9)
- added D62: LED, LED_SMD:LED_0603_1608Metric, F.Cu at (311.4, 379.5)
- added D63: LED, LED_SMD:LED_0603_1608Metric, F.Cu at (311.4, 382.1)
- added D64: LED, LED_SMD:LED_0603_1608Metric, F.Cu at (315.5, 371.7)
- added D65: LED, LED_SMD:LED_0603_1608Metric, F.Cu at (315.5, 374.3)
- added D66: LED, LED_SMD:LED_0603_1608Metric, F.Cu at (315.5, 376.9)
- added D67: LED, LED_SMD:LED_0603_1608Metric, F.Cu at (315.5, 379.5)
- added D68: LED, LED_SMD:LED_0603_1608Metric, F.Cu at (315.5, 382.1)
- added D69: 1N4148W, Diode_SMD:D_SOD-123, F.Cu at (226.8, 393.5)
- added D70: 1N4148W, Diode_SMD:D_SOD-123, F.Cu at (226.8, 396.9)
- added D71: 1N4148W, Diode_SMD:D_SOD-123, F.Cu at (226.8, 400.2)
- added D72: 1N4148W, Diode_SMD:D_SOD-123, F.Cu at (226.8, 403.6)
- added D73: 1N4148W, Diode_SMD:D_SOD-123, F.Cu at (226.8, 406.9)
- added D74: 1N4148W, Diode_SMD:D_SOD-123, F.Cu at (232.5, 370.1)
- added D75: 1N4148W, Diode_SMD:D_SOD-123, F.Cu at (232.5, 373.4)
- added D76: 1N4148W, Diode_SMD:D_SOD-123, F.Cu at (232.5, 376.8)
- added D77: 1N4148W, Diode_SMD:D_SOD-123, F.Cu at (232.5, 380.1)
- added D78: 1N4148W, Diode_SMD:D_SOD-123, F.Cu at (232.5, 383.4)
- added D79: 1N4148W, Diode_SMD:D_SOD-123, F.Cu at (232.5, 386.8)
- added D80: 1N4148W, Diode_SMD:D_SOD-123, F.Cu at (232.5, 390.1)
- added D81: 1N4148W, Diode_SMD:D_SOD-123, F.Cu at (232.5, 393.5)
- added D82: 1N4148W, Diode_SMD:D_SOD-123, F.Cu at (232.5, 396.9)
- added D83: 1N4148W, Diode_SMD:D_SOD-123, F.Cu at (232.5, 400.2)
- added JP4: Jumper_3_Bridged12, Jumper:SolderJumper-3_P1.3mm_Bridged2Bar12_RoundedPad1.0x1.5mm, F.Cu at (107.3, 283.2)
- added JP5: Jumper_2_Open, Jumpers:SolderJumper-2_P1.3mm_Open_TrianglePad1.0x1.5mm, F.Cu at (346.2, 303.5)
- added JP6: Jumper_3_Bridged12, Jumper:SolderJumper-3_P1.3mm_Bridged2Bar12_RoundedPad1.0x1.5mm, F.Cu at (26.1, 203.9)
- added R108: 10K, Resistor_SMD:R_0603_1608Metric_Pad0.98x0.95mm_HandSolder, F.Cu at (114.7, 364.8)
- added R109: 10K, Resistor_SMD:R_0603_1608Metric_Pad0.98x0.95mm_HandSolder, F.Cu at (114.7, 367.3)
- added R110: 10K, Resistor_SMD:R_0603_1608Metric_Pad0.98x0.95mm_HandSolder, F.Cu at (114.7, 369.8)
- added R111: 10K, Resistor_SMD:R_0603_1608Metric_Pad0.98x0.95mm_HandSolder, F.Cu at (114.7, 372.3)
- added R112: 10K, Resistor_SMD:R_0603_1608Metric_Pad0.98x0.95mm_HandSolder, F.Cu at (114.7, 374.8)
- added R113: 10K, Resistor_SMD:R_0603_1608Metric_Pad0.98x0.95mm_HandSolder, F.Cu at (114.7, 377.3)
- added R114: 10K, Resistor_SMD:R_0603_1608Metric_Pad0.98x0.95mm_HandSolder, F.Cu at (114.7, 379.8)
- added R115: 330R, Resistor_SMD:R_0603_1608Metric_Pad0.98x0.95mm_HandSolder, F.Cu at (302.8, 376.7)
- added R116: 330R, Resistor_SMD:R_0603_1608Metric_Pad0.98x0.95mm_HandSolder, F.Cu at (302.8, 379.2)
- added R117: 330R, Resistor_SMD:R_0603_1608Metric_Pad0.98x0.95mm_HandSolder, F.Cu at (302.8, 381.7)
- added R118: 330R, Resistor_SMD:R_0603_1608Metric_Pad0.98x0.95mm_HandSolder, F.Cu at (302.8, 384.2)
- added R119: 330R, Resistor_SMD:R_0603_1608Metric_Pad0.98x0.95mm_HandSolder, F.Cu at (307.2, 371.6)
- added R120: 330R, Resistor_SMD:R_0603_1608Metric_Pad0.98x0.95mm_HandSolder, F.Cu at (307.2, 374.2)
- added R121: 330R, Resistor_SMD:R_0603_1608Metric_Pad0.98x0.95mm_HandSolder, F.Cu at (307.2, 376.7)
- added R122: 330R, Resistor_SMD:R_0603_1608Metric_Pad0.98x0.95mm_HandSolder, F.Cu at (307.2, 379.2)
- added R123: 330R, Resistor_SMD:R_0603_1608Metric_Pad0.98x0.95mm_HandSolder, F.Cu at (307.2, 381.7)
- added R69: 4K7, Resistor_SMD:R_0402_1005Metric, F.Cu at (35.2, 197.3)
- added R70: 470R, Resistor_SMD:R_0603_1608Metric_Pad0.98x0.95mm_HandSolder, F.Cu at (302.8, 371.6)
- added R71: 10K, Resistor_SMD:R_0603_1608Metric_Pad0.98x0.95mm_HandSolder, F.Cu at (114.7, 359.8)
- added SW1: SW_Push, PaulasKiCADFootPrint:SW_PG1350, F.Cu at (125.5, 277.4)
- added SW10: SW_Push, PaulasKiCADFootPrint:SW_PG1350, F.Cu at (233.5, 277.5)
- added SW11: SW_Push, PaulasKiCADFootPrint:SW_PG1350, F.Cu at (251.5, 277.4)
- added SW12: SW_Push, PaulasKiCADFootPrint:SW_PG1350, F.Cu at (269.5, 277.4)
- added SW13: SW_Push, PaulasKiCADFootPrint:SW_PG1350, F.Cu at (242.5, 295.5)
- added SW14: SW_Push, PaulasKiCADFootPrint:SW_PG1350, F.Cu at (224.5, 295.5)
- added SW15: SW_Push, PaulasKiCADFootPrint:SW_PG1350, F.Cu at (260.5, 259.5)
- added SW16: SW_Push, PaulasKiCADFootPrint:SW_PG1350, F.Cu at (278.5, 259.5)
- added SW17: SW_Push, PaulasKiCADFootPrint:SW_PG1350, F.Cu at (116.5, 259.4)
- added SW18: SW_Push, PaulasKiCADFootPrint:SW_PG1350, F.Cu at (206.5, 259.5)
- added SW19: SW_Push, PaulasKiCADFootPrint:SW_PG1350, F.Cu at (170.5, 259.4)
- added SW2: SW_Push, PaulasKiCADFootPrint:SW_PG1350, F.Cu at (206.5, 295.5)
- added SW20: SW_Push, PaulasKiCADFootPrint:SW_PG1350, F.Cu at (134.5, 295.5)
- added SW21: SW_Push, PaulasKiCADFootPrint:SW_PG1350, F.Cu at (143.5, 277.5)
- added SW22: SW_Push, PaulasKiCADFootPrint:SW_PG1350, F.Cu at (269.5, 241.4)
- added SW23: SW_Push, PaulasKiCADFootPrint:SW_PG1350, F.Cu at (188.5, 259.5)
- added SW24: SW_Push, PaulasKiCADFootPrint:SW_PG1350, F.Cu at (107.5, 241.4)
- added SW25: SW_Push, PaulasKiCADFootPrint:SW_PG1350, F.Cu at (224.5, 259.5)
- added SW26: SW_Push, PaulasKiCADFootPrint:SW_PG1350, F.Cu at (125.5, 241.4)
- added SW27: SW_Push, PaulasKiCADFootPrint:SW_PG1350, F.Cu at (188.5, 295.5)
- added SW28: SW_Push, PaulasKiCADFootPrint:SW_PG1350, F.Cu at (143.5, 241.4)
- added SW29: SW_Push, PaulasKiCADFootPrint:SW_PG1350, F.Cu at (134.5, 259.4)
- added SW3: SW_Push, PaulasKiCADFootPrint:SW_PG1350, F.Cu at (170.5, 295.5)
- added SW30: SW_Push, PaulasKiCADFootPrint:SW_PG1350, F.Cu at (161.5, 241.4)
- added SW31: SW_Push, PaulasKiCADFootPrint:SW_PG1350, F.Cu at (152.5, 295.5)
- added SW32: SW_Push, PaulasKiCADFootPrint:SW_PG1350, F.Cu at (179.5, 241.4)
- added SW33: SW_Push, PaulasKiCADFootPrint:SW_PG1350, F.Cu at (197.5, 241.4)
- added SW34: SW_Push, PaulasKiCADFootPrint:SW_PG1350, F.Cu at (287.5, 277.4)
- added SW35: SW_Push, PaulasKiCADFootPrint:SW_PG1350, F.Cu at (215.5, 241.4)
- added SW36: SW_Push, PaulasKiCADFootPrint:SW_PG1350, F.Cu at (305.5, 277.5)
- added SW37: SW_Push, PaulasKiCADFootPrint:SW_PG1350, F.Cu at (233.5, 241.4)
- added SW38: SW_Push, PaulasKiCADFootPrint:SW_PG1350, F.Cu at (323.5, 277.5)
- added SW39: SW_Push, PaulasKiCADFootPrint:SW_PG1350, F.Cu at (251.5, 241.4)
- added SW4: SW_Push, PaulasKiCADFootPrint:SW_PG1350, F.Cu at (161.5, 277.5)
- added SW40: SW_Push, PaulasKiCADFootPrint:SW_PG1350, F.Cu at (260.5, 295.5)
- added SW41: SW_Push, PaulasKiCADFootPrint:SW_PG1350, F.Cu at (287.5, 241.4)
- added SW42: SW_Push, PaulasKiCADFootPrint:SW_PG1350, F.Cu at (278.5, 295.5)
- added SW43: SW_Push, PaulasKiCADFootPrint:SW_PG1350, F.Cu at (305.5, 241.4)
- added SW44: SW_Push, PaulasKiCADFootPrint:SW_PG1350, F.Cu at (296.5, 295.5)
- added SW45: SW_Push, PaulasKiCADFootPrint:SW_PG1350, F.Cu at (296.5, 259.5)
- added SW46: SW_Push, PaulasKiCADFootPrint:SW_PG1350, F.Cu at (116.5, 295.4)
- added SW47: SW_Push, PaulasKiCADFootPrint:SW_PG1350, F.Cu at (314.5, 259.4)
- added SW48: SW_Push, PaulasKiCADFootPrint:SW_PG1350, F.Cu at (175.0, 313.5)
- added SW49: SW_Push, PaulasKiCADFootPrint:SW_PG1350, F.Cu at (305.5, 313.4)
- added SW5: SW_Push, PaulasKiCADFootPrint:SW_PG1350, F.Cu at (152.5, 259.4)
- added SW50: SW_Push, PaulasKiCADFootPrint:SW_PG1350, F.Cu at (323.5, 313.5)
- added SW51: SW_Push, PaulasKiCADFootPrint:SW_PG1350, F.Cu at (287.5, 313.5)
- added SW52: SW_Push, PaulasKiCADFootPrint:SW_PG1350, F.Cu at (341.5, 313.5)
- added SW53: SW_Push, PaulasKiCADFootPrint:SW_PG1350, F.Cu at (323.5, 241.4)
- added SW54: SW_Push, PaulasKiCADFootPrint:SW_PG1350, F.Cu at (125.5, 313.5)
- added SW55: SW_Push, PaulasKiCADFootPrint:SW_PG1350, F.Cu at (341.6, 268.5)
- added SW57: SW_Push, PaulasKiCADFootPrint:SW_PG1350, F.Cu at (98.5, 259.4)
- added SW58: SW_Push, PaulasKiCADFootPrint:SW_PG1350, F.Cu at (98.5, 295.4)
- added SW59: SW_Push, PaulasKiCADFootPrint:SW_PG1350, F.Cu at (98.5, 313.4)
- added SW6: SW_Push, PaulasKiCADFootPrint:SW_PG1350, F.Cu at (179.5, 277.5)
- added SW60: SW_Push, PaulasKiCADFootPrint:SW_PG1350, F.Cu at (238.0, 313.4)
- added SW61: SW_Push, PaulasKiCADFootPrint:SW_PG1350, F.Cu at (206.5, 313.5)
- added SW65: SW_Push, PaulasKiCADFootPrint:SW_PG1350, F.Cu at (314.5, 295.5)
- added SW7: SW_Push, PaulasKiCADFootPrint:SW_PG1350, F.Cu at (197.5, 277.4)
- added SW8: SW_Push, PaulasKiCADFootPrint:SW_PG1350, F.Cu at (215.5, 277.5)
- added SW9: SW_Push, PaulasKiCADFootPrint:SW_PG1350, F.Cu at (242.5, 259.5)
- C40, C49: footprint Capacitor_SMD:C_0603_1608Metric -> Capacitor_SMD:C_0805_2012Metric
- C48: footprint Capacitor_SMD:C_0603_1608Metric -> Capacitor_SMD:C_0402_1005Metric
- C56, C57, C58, C59, J12, J13, J3, J6, LS1, S1, S2, U13, VR1, X1: moved to F.Cu
- C60: value 10uF NP -> 100nF; footprint Capacitor_SMD:C_0805_2012Metric -> Capacitor_SMD:C_0402_1005Metric
- C61: value 10uF NP -> 47uF; footprint Capacitor_SMD:C_0805_2012Metric -> Capacitor_SMD:C_1206_3216Metric
- C64, C66: footprint Capacitor_SMD:C_0402_1005Metric -> Capacitor_SMD:C_0805_2012Metric
- C65: value 100nF -> 47uF; footprint Capacitor_SMD:C_0402_1005Metric -> Capacitor_SMD:C_1206_3216Metric
- D12, D13: value 1N4148 -> 1N4148W; footprint Diode_THT:D_DO-35_SOD27_P7.62mm_Horizontal -> Diode_SMD:D_SOD-123
- D14: value B5819W SL -> 1N4148W
- D17: value 1N4148 -> LED; footprint Diode_THT:D_DO-35_SOD27_P7.62mm_Horizontal -> LED_THT:LED_D5.0mm
- J10: value Conn_02x05_Odd_Even -> Conn_02x20_Odd_Even; footprint Connector_PinHeader_2.54mm:PinHeader_2x05_P2.54mm_Vertical -> Connector_PinHeader_2.54mm:PinHeader_2x20_P2.54mm_Horizontal; moved to B.Cu
- J5: footprint Connector_PinHeader_2.54mm:PinHeader_2x20_P2.54mm_Vertical -> FFC3B07-40-T:GCT_FFC3B07-40-T; moved to F.Cu
- J7: value Conn_01x02 -> Conn_02x05_Odd_Even; footprint Connector_PinHeader_2.54mm:PinHeader_1x02_P2.54mm_Horizontal -> Connector_PinHeader_2.54mm:PinHeader_2x05_P2.54mm_Horizontal
- Q2: value IRLML6402 -> STL9P3LLH6; footprint Package_TO_SOT_SMD:SOT-23 -> STL9P3LLH6:STL20N6F7
- R107: value 10K -> 330R; footprint Resistor_SMD:R_0402_1005Metric -> Resistor_SMD:R_0603_1608Metric_Pad0.98x0.95mm_HandSolder
- R74: value 10k -> 100K
- R82: value 3K3 -> 10K; footprint Resistor_SMD:R_0402_1005Metric -> Resistor_SMD:R_0603_1608Metric_Pad0.98x0.95mm_HandSolder
- U12: value W65C51NxP -> ATmega644P-20A; footprint Package_DIP:DIP-28_W15.24mm -> Package_QFP:TQFP-44_10x10mm_P0.8mm
- U14: value AMS1117-3.3 -> TXS0102DCT; footprint Package_TO_SOT_SMD:SOT-223-3_TabPin2 -> Package_SO:SSOP-8_2.95x2.8mm_P0.65mm
- U15: value TXS0102DCT -> 74HCT138; footprint Package_SO:SSOP-8_2.95x2.8mm_P0.65mm -> Package_SO:SSOP-16_5.3x6.2mm_P0.65mm
- moved J10 478.4 mm to (452.5, 469.8), turned to -90 degrees
- moved C44 468.6 mm to (483.8, 518.0)
- moved C43 467.3 mm to (488.1, 517.7)
- moved D19 459.1 mm to (483.2, 511.1)
- moved D21 459.1 mm to (483.2, 514.7)
- moved C62 372.1 mm to (134.6, 401.2)
- moved C63 372.1 mm to (134.6, 403.2)
- moved C40 366.3 mm to (119.1, 377.8)
- moved R97 364.2 mm to (134.6, 391.3)
- moved R98 364.2 mm to (134.6, 393.3)
- moved R101 364.2 mm to (134.6, 395.3)
- moved R104 364.2 mm to (134.6, 397.3)
- moved Q2 364.1 mm to (138.5, 376.2)
- moved R105 363.1 mm to (131.2, 401.6)
- moved R106 363.1 mm to (131.2, 404.1)
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Connections:
- C38 pad 1: /60FAKE50/VUSB -> +5V
- C40 pad 1: Net-(J7-Pin_2) -> +5V
- C40 pad 2: Net-(Q2-G) -> GND
- C41 pad 1: /60FAKE50/VUSB -> +5V
- C42 pad 1: /60FAKE50/VUSB -> +5V
- C49 pad 1: +5V -> AVR_nRST
- C60 pad 1: +5V -> +3.3V
- C64 pad 1: AVR_nRST -> +5V
- D12 pad 1: Net-(D12-K) -> /Keyboard IF/KeyMatrix/COL0
- D12 pad 2: nRAMDISABLE -> Net-(D12-A)
- D13 pad 1: Net-(D13-K) -> /Keyboard IF/KeyMatrix/COL0
- D13 pad 2: nROMDISABLE -> Net-(D13-A)
- D14 pad 1: /60FAKE50/VUSB -> /Keyboard IF/KeyMatrix/COL0
- D14 pad 2: +5V -> Net-(D14-A)
- D17 pad 1: Net-(D17-K) -> KEYLED0
- D17 pad 2: nIRQ -> Net-(D17-A)
- IC1 pad 28: Net-(IC1-I/O_21) -> unconnected-(IC1-I/O_21-Pad28)
- IC1 pad 29: Net-(IC1-I/O_22) -> unconnected-(IC1-I/O_22-Pad29)
- IC1 pad 30: Net-(IC1-I/O_23) -> KEYLED_PWM
- IC1 pad 31: Net-(IC1-I/O_24) -> MODEM_nRST
- IC1 pad 32: Net-(IC1-I/O_25) -> MODEM_EN
- IC1 pad 33: /Glue_Addr/MODEM_RnW -> MODEM_nCS
- IC1 pad 35: /Glue_Addr/MODEM_nCS -> MODEM_nCS
- IC1 pad 61: /ExpansionSlot0/CPLD_nDIS -> unconnected-(IC1-I/O_47-Pad61)
- IC1 pad 71: nROMDISABLE -> unconnected-(IC1-I/O_55-Pad71)
- IC1 pad 72: nRAMDISABLE -> unconnected-(IC1-I/O_56-Pad72)
- IC1 pad 79: nOSC_DISABLE -> unconnected-(IC1-I/O_61-Pad79)
- IC1 pad 85: SLOT_OSC -> unconnected-(IC1-I/O/GCLK3-Pad85)
- J10 pad 1: AVR_TCK -> +5V
- J10 pad 10: GND -> /A5
- J10 pad 2: GND -> +5V
- J10 pad 3: AVR_TDO -> +5V
- J10 pad 5: AVR_TMS -> /A0
- J10 pad 6: AVR_nRST -> /A1
- J10 pad 7: unconnected-(J10-Pin_7-Pad7) -> /A2
- J10 pad 8: unconnected-(J10-Pin_8-Pad8) -> /A3
- J10 pad 9: AVR_TDI -> /A4
- J7 pad 1: +5V -> AVR_TCK
- J7 pad 2: Net-(J7-Pin_2) -> GND
- Q2 pad 1: Net-(Q2-G) -> +5V
- Q2 pad 2: /60FAKE50/VUSB -> +5V
- Q2 pad 3: Net-(J7-Pin_2) -> +5V
- R101 pad 2: Net-(U15-B1) -> Net-(U14-B1)
- R102 pad 1: /Modem/ESP01_nRST -> MODEM_nRST
- R104 pad 2: Net-(U15-B2) -> Net-(U14-B2)
- R105 pad 1: Net-(U15-B1) -> Net-(U14-B1)
- R105 pad 2: /Modem/RX_5V -> MODEM_SER_IN
- R106 pad 1: Net-(U15-B2) -> Net-(U14-B2)
- R106 pad 2: /Modem/TX_5V -> MODEM_SER_OUT
- R107 pad 1: +5V -> GND
- R107 pad 2: AVR_nRST -> Net-(D56-K)
- R14 pad 2: nOSC_DISABLE -> Net-(X1-EN)
- R72 pad 2: /60FAKE50/VUSB -> GND
- R73 pad 2: /60FAKE50/VUSB -> +5V
- R74 pad 1: Net-(U10-~{PWREN}) -> +5V
- R74 pad 2: Net-(Q2-G) -> KEYLED_PWM
- R82 pad 2: Net-(X2-EN) -> ROW0
- R87 pad 1: /Glue_Addr/MODEM_nCS -> MODEM_nCS
- R95 pad 2: /Modem/BATTMON -> /Keyboard IF/BATTMON
- R97 pad 2: /Modem/TX_3V3 -> /Keyboard IF/Modem/TX_3V3
- R98 pad 2: /Modem/RX_3V3 -> /Keyboard IF/Modem/RX_3V3
- R99 pad 1: /Modem/ESP01_EN -> MODEM_EN
- U10 pad 20: /60FAKE50/VUSB -> +5V
- U10 pad 4: /60FAKE50/VUSB -> +5V
- U12 pad 1: GND -> ROW5
- U12 pad 10: Net-(J14-Pin_2) -> MODEM_SER_OUT
- U12 pad 11: unconnected-(U12-~{DTR}-Pad11) -> MODEM_nCS
- U12 pad 12: Net-(J14-Pin_3) -> ACIA_nCS
- U12 pad 13: /A0 -> nRES
- U12 pad 14: /A1 -> Net-(U12-PD5)
- U12 pad 15: +5V -> Net-(U12-PD6)
- U12 pad 16: GND -> Net-(U12-PD7)
- U12 pad 17: GND -> +5V
- U12 pad 18: /D0 -> GND
- U12 pad 19: /D1 -> /A0
- U12 pad 2: +5V -> ROW6
- U12 pad 20: /D2 -> RnW
- U12 pad 21: /D3 -> AVR_TCK
- U12 pad 22: /D4 -> AVR_TMS
- U12 pad 23: /D5 -> AVR_TDO
- U12 pad 24: /D6 -> AVR_TDI
- U12 pad 25: /D7 -> KEYLED0
- U12 pad 26: Net-(D17-K) -> /D7
- U12 pad 27: CLK -> +5V
- U12 pad 28: RnW -> GND
- U12 pad 3: ACIA_nCS -> ROW7
- U12 pad 4: nRES -> AVR_nRST
- U12 pad 5: unconnected-(U12-RxC-Pad5) -> +5V
- U12 pad 6: Net-(U12-XTAL1) -> GND
- U12 pad 8: unconnected-(U12-~{RTS}-Pad8) -> Net-(U12-XTAL1)
- U12 pad 9: GND -> MODEM_SER_IN
- U13 pad 4: /Modem/RX_3V3 -> /Keyboard IF/Modem/RX_3V3
- U13 pad 5: /Modem/TX_3V3 -> /Keyboard IF/Modem/TX_3V3
- U14 pad 1: GND -> Net-(U14-B2)
- U14 pad 2: +3.3V -> GND
- U14 pad 3: +5V -> +3.3V
- U15 pad 1: Net-(U15-B2) -> Net-(U12-PD5)
- U15 pad 2: GND -> Net-(U12-PD6)
- U15 pad 3: +3.3V -> Net-(U12-PD7)
- U15 pad 4: /Modem/RX_3V3 -> GND
- U15 pad 5: /Modem/TX_3V3 -> GND
- U15 pad 6: +3.3V -> +5V
- U15 pad 7: +5V -> /Keyboard IF/KeyMatrix/COL7
- U15 pad 8: Net-(U15-B1) -> GND
- X1 pad 1: nOSC_DISABLE -> Net-(X1-EN)
- Y1 pad 3: Net-(U16-XTAL1) -> Net-(U12-XTAL1)
Other:
- board size 190 x 175 mm -> 280 x 180 mm
- board text added: "#"
- board text added: "-"
- board text added: "/"
- board text added: "0"
- board text added: "1"
- board text added: "1N4148W"
- board text added: "2"
- board text added: "6"
- board text added: "7"
- board text added: "8"
- board text added: "9"
- board text added: ";"
- board text added: "<"
- board text added: "="
- board text added: ">"
- board text added: "@"
- board text added: "A"
- board text added: "ARROW PWM"
- board text added: "B"
- board text added: "BREAK"
- board text added: "C"
- board text added: "CAPS"
- board text added: "CTRL"
- board text added: "D"
- board text added: "DELETE"
- board text added: "DOWN"
- board text added: "E"
- board text added: "ENTER"
- board text added: "F"
- board text added: "G"
- board text added: "H"
- board text added: "I"
- board text added: "J"
- board text added: "K"
- board text added: "L"
- board text added: "LEFT"
- board text added: "M"
- board text added: "N"
- board text added: "O"
- board text added: "ON"
- board text added: "P"
- board text added: "PWM"
- board text added: "Q"
- board text added: "R"
- board text added: "RIGHT"
- board text added: "S"
- board text added: "SHIFT"
- board text added: "SPACE"
- board text added: "T"
- board text added: "TAB"
- board text added: "U"
- board text added: "UP"
- board text added: "V"
- board text added: "W"
- board text added: "X"
- board text added: "Y"
- board text added: "Z"
- board text added: "["
- board text added: "\"
- board text added: "]"

Commit message: Work on parts placement, remove excess LEDs
Parts:
- moved C43 430.5 mm to (558.2, 93.0)
- moved C44 430.5 mm to (554.0, 93.2)
- moved D19 430.5 mm to (553.3, 86.4)
- moved D21 430.5 mm to (553.3, 90.0)
- moved J10 408.3 mm to (515.7, 66.5)
- moved H2 388.1 mm to (355.0, 314.0)
- moved FOX1 373.5 mm to (350.0, 340.0)
- moved H9 350.4 mm to (306.0, 345.0)
- moved H7 350.2 mm to (356.0, 256.0)
- moved H4 328.7 mm to (356.0, 174.0)
- moved H6 288.3 mm to (206.0, 345.0)
- moved H1 224.4 mm to (85.0, 313.0)
- moved H5 217.0 mm to (216.0, 226.0)
- moved C66 211.2 mm to (322.6, 330.4)
- moved Q2 189.5 mm to (323.2, 333.9), turned to -90 degrees
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Other:
- outline, holes or cut-outs redrawn
- board text added: "NOT SURE IF I CAN FIT THIS IN"
