File: Schematics/MainBoard/keyleds.kicad_sch (KiCad schematic)
At the start: 24 parts

Commit message: Work on PCB
Parts:
- R107, R115, R116, R117, R118, R119, R120, R121, R122, R123, R70: footprint Resistor_SMD:R_0603_1608Metric_Pad0.98x0.95mm_HandSolder -> Resistor_SMD:R_0402_1005Metric
Changed lines of the file:
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@@
 			)
 		)
-		(property "Footprint" "Resistor_SMD:R_0603_1608Metric_Pad0.98x0.95mm_HandSolder"
+		(property "Footprint" "Resistor_SMD:R_0402_1005Metric"
 			(at 138.43 82.042 90)
 			(effects
@@
 			)
 		)
-		(property "Footprint" "Resistor_SMD:R_0603_1608Metric_Pad0.98x0.95mm_HandSolder"
+		(property "Footprint" "Resistor_SMD:R_0402_1005Metric"
 			(at 200.66 82.042 90)
 			(effects
@@
 			)
 		)
-		(property "Footprint" "Resistor_SMD:R_0603_1608Metric_Pad0.98x0.95mm_HandSolder"
+		(property "Footprint" "Resistor_SMD:R_0402_1005Metric"
 			(at 138.43 56.642 90)
 			(effects
@@
 			)
 		)
-		(property "Footprint" "Resistor_SMD:R_0603_1608Metric_Pad0.98x0.95mm_HandSolder"
+		(property "Footprint" "Resistor_SMD:R_0402_1005Metric"
 			(at 138.43 127.762 90)
 			(effects
@@
 			)
 		)
-		(property "Footprint" "Resistor_SMD:R_0603_1608Metric_Pad0.98x0.95mm_HandSolder"
+		(property "Footprint" "Resistor_SMD:R_0402_1005Metric"
 			(at 138.43 99.822 90)
 			(effects
@@
 			)
 		)
-		(property "Footprint" "Resistor_SMD:R_0603_1608Metric_Pad0.98x0.95mm_HandSolder"
+		(property "Footprint" "Resistor_SMD:R_0402_1005Metric"
 			(at 138.43 69.342 90)
 			(effects
@@
 			)
 		)
-		(property "Footprint" "Resistor_SMD:R_0603_1608Metric_Pad0.98x0.95mm_HandSolder"
+		(property "Footprint" "Resistor_SMD:R_0402_1005Metric"
 			(at 113.03 165.862 90)
 			(effects
@@
 			)
 		)
-		(property "Footprint" "Resistor_SMD:R_0603_1608Metric_Pad0.98x0.95mm_HandSolder"
+		(property "Footprint" "Resistor_SMD:R_0402_1005Metric"
 			(at 138.43 112.522 90)
 			(effects
@@
 			)
 		)
-		(property "Footprint" "Resistor_SMD:R_0603_1608Metric_Pad0.98x0.95mm_HandSolder"
+		(property "Footprint" "Resistor_SMD:R_0402_1005Metric"
 			(at 200.66 69.342 90)
 			(effects
@@
 			)
 		)
-		(property "Footprint" "Resistor_SMD:R_0603_1608Metric_Pad0.98x0.95mm_HandSolder"
+		(property "Footprint" "Resistor_SMD:R_0402_1005Metric"
 			(at 200.66 56.642 90)
 			(effects
@@
 			)
 		)
-		(property "Footprint" "Resistor_SMD:R_0603_1608Metric_Pad0.98x0.95mm_HandSolder"
+		(property "Footprint" "Resistor_SMD:R_0402_1005Metric"
 			(at 200.66 43.942 90)
 			(effects

Commit message: Updates based on production files for JLC
Parts:
- D17, JP5: now not fitted
- D56, D60, D61, D62, D63, D64, D65, D66, D67, D68: LCSC C3030991 -> C2286
- JP4: LCSC (none) -> DNF; now not fitted
- R107, R115, R116, R117, R118, R119, R120, R121, R122, R123: LCSC DNF -> C25104
- R70: LCSC DNF -> C25117
Changed lines of the file:
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@@
 			)
 		)
-		(property "LCSC" "C3030991"
+		(property "LCSC" "C2286"
 			(at 125.73 101.6 0)
 			(effects
@@
 			)
 		)
-		(property "LCSC" "DNF"
+		(property "LCSC" "C25104"
 			(at 138.43 83.82 90)
 			(effects
@@
 			)
 		)
-		(property "LCSC" "C3030991"
+		(property "LCSC" "C2286"
 			(at 187.96 71.12 0)
 			(effects
@@
 			)
 		)
-		(property "LCSC" "C3030991"
+		(property "LCSC" "C2286"
 			(at 187.96 45.72 0)
 			(effects
@@
 			)
 		)
-		(property "LCSC" "C3030991"
+		(property "LCSC" "C2286"
 			(at 187.96 58.42 0)
 			(effects
@@
 			)
 		)
-		(property "LCSC" "DNF"
+		(property "LCSC" "C25104"
 			(at 200.66 83.82 90)
 			(effects
@@
 			)
 		)
-		(property "LCSC" "C3030991"
+		(property "LCSC" "C2286"
 			(at 125.73 129.54 0)
 			(effects
@@
 		(in_bom yes)
 		(on_board yes)
-		(dnp no)
+		(dnp yes)
 		(fields_autoplaced yes)
 		(property "Reference" "D17"
@@
 			)
 		)
-		(property "LCSC" "DNF"
+		(property "LCSC" "C25104"
 			(at 138.43 58.42 90)
 			(effects
@@
 		(in_bom no)
 		(on_board yes)
-		(dnp no)
+		(dnp yes)
 		(fields_autoplaced yes)
 		(property "Reference" "JP4"
@@
 			)
 		)
+		(property "LCSC" "DNF"
+			(at 92.71 146.05 0)
+			(effects
+				(font
+					(size 1.27 1.27)
+				)
+				(hide yes)
+			)
+		)
 		(pin "3"
 		)
@@
 			)
 		)
-		(property "LCSC" "DNF"
+		(property "LCSC" "C25104"
 			(at 138.43 129.54 90)
 			(effects
@@
 		(in_bom yes)
 		(on_board yes)
-		(dnp no)
+		(dnp yes)
 		(fields_autoplaced yes)
 		(property "Reference" "JP5"
@@
 			)
 		)
-		(property "LCSC" "DNF"
+		(property "LCSC" "C25104"
 			(at 138.43 101.6 90)
 			(effects
@@
 			)
 		)
-		(property "LCSC" "C3030991"
+		(property "LCSC" "C2286"
 			(at 125.73 114.3 0)
 			(effects
@@
 			)
 		)
-		(property "LCSC" "DNF"
+		(property "LCSC" "C25104"
 			(at 138.43 71.12 90)
 			(effects
@@
 			)
 		)
-		(property "LCSC" "C3030991"
+		(property "LCSC" "C2286"
 			(at 125.73 58.42 0)
 			(effects
@@
 			)
 		)
-		(property "LCSC" "DNF"
+		(property "LCSC" "C25117"
 			(at 113.03 167.64 90)
 			(effects
@@
 			)
 		)
-		(property "LCSC" "C3030991"
+		(property "LCSC" "C2286"
 			(at 125.73 71.12 0)
 			(effects
@@
 			)
 		)
-		(property "LCSC" "DNF"
+		(property "LCSC" "C25104"
 			(at 138.43 114.3 90)
 			(effects
@@
 			)
 		)
-		(property "LCSC" "C3030991"
+		(property "LCSC" "C2286"
 			(at 125.73 83.82 0)
 			(effects
@@
 			)
 		)
-		(property "LCSC" "DNF"
+		(property "LCSC" "C25104"
 			(at 200.66 71.12 90)
 			(effects
@@
 			)
 		)
-		(property "LCSC" "DNF"
+		(property "LCSC" "C25104"
 			(at 200.66 58.42 90)
 			(effects
@@
 			)
 		)
-		(property "LCSC" "C3030991"
+		(property "LCSC" "C2286"
 			(at 187.96 83.82 0)
 			(effects
@@
 			)
 		)
-		(property "LCSC" "DNF"
+		(property "LCSC" "C25104"
 			(at 200.66 45.72 90)
 			(effects
