File: Schematics/MainBoard/nanoSwinSID.kicad_sch (KiCad schematic)
At the start: 14 parts, among them J11 Conn_02x03_Odd_Even, U18 ATmega88PA-AU, Y2 ECS-3961-320-AU-TR

Commit message: Updates based on production files for JLC
Parts:
- C70, C72: LCSC C113803 -> C307331
- C71: LCSC (none) -> C1620
- J11, JP7: LCSC (none) -> DNF; now not fitted
- R124: LCSC (none) -> C4190
- R125: value 4.7k -> 4K7; LCSC (none) -> C25900
- R24, R61: LCSC (none) -> DNF
- R90: LCSC (none) -> C11702
- R96: LCSC (none) -> 0402
Changed lines of the file:
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@@
+			)
+		)
+		(property "LCSC" "C11702"
+			(at 154.94 67.31 90)
+			(effects
+				(font
+					(size 1.27 1.27)
+				)
+				(hide yes)
 			)
 		)
@@
 		(in_bom yes)
 		(on_board yes)
-		(dnp no)
+		(dnp yes)
 		(property "Reference" "JP7"
 			(at 130.81 51.7144 0)
@@
 			)
 		)
+		(property "LCSC" "DNF"
+			(at 130.81 58.42 0)
+			(effects
+				(font
+					(size 1.27 1.27)
+				)
+				(hide yes)
+			)
+		)
 		(pin "1"
 		)
@@
 		(in_bom yes)
 		(on_board yes)
-		(dnp no)
+		(dnp yes)
 		(property "Reference" "J11"
 			(at 37.465 88.265 0)
@@
 					(size 1.27 1.27)
 				)
+			)
+		)
+		(property "LCSC" "DNF"
+			(at 36.195 93.98 0)
+			(effects
+				(font
+					(size 1.27 1.27)
+				)
+				(hide yes)
 			)
 		)
@@
 			)
 		)
+		(property "LCSC" "DNF"
+			(at 78.74 63.5 0)
+			(effects
+				(font
+					(size 1.27 1.27)
+				)
+				(hide yes)
+			)
+		)
 		(pin "1"
 		)
@@
 			)
 		)
+		(property "LCSC" "C4190"
+			(at 165.735 67.31 90)
+			(effects
+				(font
+					(size 1.27 1.27)
+				)
+				(hide yes)
+			)
+		)
 		(pin "1"
 		)
@@
 			)
 		)
+		(property "LCSC" "0402"
+			(at 154.305 74.93 90)
+			(effects
+				(font
+					(size 1.27 1.27)
+				)
+				(hide yes)
+			)
+		)
 		(pin "1"
 		)
@@
 					(size 1.27 1.27)
 				)
+			)
+		)
+		(property "LCSC" "C1620"
+			(at 160.02 80.01 0)
+			(effects
+				(font
+					(size 1.27 1.27)
+				)
+				(hide yes)
 			)
 		)
@@
 			)
 		)
-		(property "LCSC" "C113803"
+		(property "LCSC" "C307331"
 			(at 62.23 50.8 0)
 			(effects
@@
 			)
 		)
-		(property "Value" "4.7k"
+		(property "Value" "4K7"
 			(at 177.8 62.865 0)
 			(effects
@@
 					(size 1.27 1.27)
 				)
+			)
+		)
+		(property "LCSC" "C25900"
+			(at 173.99 61.595 0)
+			(effects
+				(font
+					(size 1.27 1.27)
+				)
+				(hide yes)
 			)
 		)
@@
 			)
 		)
+		(property "LCSC" "DNF"
+			(at 142.24 81.28 0)
+			(effects
+				(font
+					(size 1.27 1.27)
+				)
+				(hide yes)
+			)
+		)
 		(pin "1"
 		)
@@
 			)
 		)
-		(property "LCSC" "C113803"
+		(property "LCSC" "C307331"
 			(at 87.63 167.64 0)
 			(effects
