File: Schematics/MainBoard/CompactFlash.kicad_sch (KiCad schematic)
At the start: 10 parts, among them J8 Conn_02x26_Top_Bottom

Commit message: Work on PCB
Parts:
- C50: footprint Capacitor_SMD:C_0603_1608Metric -> Capacitor_SMD:C_0402_1005Metric
Changed lines of the file:
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@@
 			)
 		)
-		(property "Footprint" "Capacitor_SMD:C_0603_1608Metric"
+		(property "Footprint" "Capacitor_SMD:C_0402_1005Metric"
 			(at 91.7448 72.39 0)
 			(effects

Commit message: Updates based on production files for JLC
Parts:
- C50: LCSC C113803 -> C307331
- D11: LCSC DNF -> C2296
- J8, R75: now not fitted
Changed lines of the file:
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@@
 			)
 		)
-		(property "LCSC" "C113803"
+		(property "LCSC" "C307331"
 			(at 92.71 68.58 0)
 			(effects
@@
 		(in_bom yes)
 		(on_board yes)
-		(dnp no)
+		(dnp yes)
 		(fields_autoplaced yes)
 		(property "Reference" "J8"
@@
 		(in_bom yes)
 		(on_board yes)
-		(dnp no)
+		(dnp yes)
 		(property "Reference" "R75"
 			(at 108.204 85.344 90)
@@
 			)
 		)
-		(property "LCSC" "DNF"
+		(property "LCSC" "C2296"
 			(at 209.55 92.71 0)
 			(effects
