File: Schematics/MainBoard/MainBoard.kicad_sch (KiCad schematic)
At the start: 39 parts, among them U1 TC1232, U2 W65C02S6TQG-14, U3 IS62C256AL, U4 IS62C256AL, U5 SST39SF010

Commit message: Updates based on production files for JLC
Parts:
- C1, C2, C3, C4, C5, C53: LCSC C113803 -> C307331
- C59: LCSC DNP -> C49332976
- S2, U1, U2, U5: now not fitted
- U3, U4: LCSC DNF -> C14323
Changed lines of the file:
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@@
 			)
 		)
-		(property "LCSC" "DNF"
+		(property "LCSC" "C14323"
 			(at 328.93 58.42 0)
 			(effects
@@
 		(in_bom yes)
 		(on_board yes)
-		(dnp no)
+		(dnp yes)
 		(fields_autoplaced yes)
 		(property "Reference" "U2"
@@
 			)
 		)
-		(property "LCSC" "DNP"
+		(property "LCSC" "C49332976"
 			(at 83.82 142.24 0)
 			(effects
@@
 			)
 		)
-		(property "LCSC" "C113803"
+		(property "LCSC" "C307331"
 			(at 54.61 265.43 0)
 			(effects
@@
 			)
 		)
-		(property "LCSC" "C113803"
+		(property "LCSC" "C307331"
 			(at 31.75 265.43 0)
 			(effects
@@
 			)
 		)
-		(property "LCSC" "C113803"
+		(property "LCSC" "C307331"
 			(at 88.9 265.43 0)
 			(effects
@@
 			)
 		)
-		(property "LCSC" "C113803"
+		(property "LCSC" "C307331"
 			(at 25.4 265.43 0)
 			(effects
@@
 			)
 		)
-		(property "LCSC" "DNF"
+		(property "LCSC" "C14323"
 			(at 328.93 119.38 0)
 			(effects
@@
 		(in_bom yes)
 		(on_board yes)
-		(dnp no)
+		(dnp yes)
 		(property "Reference" "S2"
 			(at 27.178 183.134 0)
@@
 		(in_bom yes)
 		(on_board yes)
-		(dnp no)
+		(dnp yes)
 		(property "Reference" "U5"
 			(at 337.185 158.75 0)
@@
 			)
 		)
-		(property "LCSC" "C113803"
+		(property "LCSC" "C307331"
 			(at 60.96 265.43 0)
 			(effects
@@
 		(in_bom yes)
 		(on_board yes)
-		(dnp no)
+		(dnp yes)
 		(fields_autoplaced yes)
 		(property "Reference" "U1"
@@
 			)
 		)
-		(property "LCSC" "C113803"
+		(property "LCSC" "C307331"
 			(at 82.55 265.43 0)
 			(effects

Commit message: Add some comments to schematic, update README, start on GLUE
Add some comments to schematic, update README, start on GLUE
Other:
- sheet Display Connector ports: added DISP_E; removed DISP_EN
- sheet Glue_Addr ports: added DISP_E; removed DISP_EN
